File: hardware/sdc-ntc-emulator/sdc-ntc-emulator.kicad_sch (KiCad schematic)
At the start: 37 parts, among them J1 DevKit J1, J2 DevKit J3, J3 5V IN (RAC03), J4 SDC VE1 / GND, K1 G5V-2-H1 5VDC, Q1 AO3400A, Q2 AO3401A, U1 ISO1540, U2 AD5272BRMZ-50

Commit message: PCB rev 3: TMR 1-0511 isolated supply, DigiKey-verified BOM
- PS1 Traco TMR 1-0511 (SIP-6) replaces the TEM 2-0511; straight isolation gap >= 1.40 mm
- Parts that were obsolete, backordered or not stocked at DigiKey replaced by stocked equivalents
- DigiKey upload file carries DigiKey part numbers; quantities follow DigiKey price breaks, spares only where useful

Co-Authored-By: Claude Opus 5.5 <noreply@anthropic.com>
Parts:
- removed R8: 270R 0.6W, Resistor_THT:R_Axial_DIN0207_L6.3mm_D2.5mm_P10.16mm_Horizontal, symbol Device:R
- added C10, C11: 100nF, Capacitor_SMD:C_0805_2012Metric_Pad1.18x1.45mm_HandSolder, symbol Device:C
- added D3: green, LED_SMD:LED_0805_2012Metric_Pad1.15x1.40mm_HandSolder, symbol Device:LED
- added D4: yellow, LED_SMD:LED_0805_2012Metric_Pad1.15x1.40mm_HandSolder, symbol Device:LED
- added J5: SDC SERVICE, Connector_JST:JST_XH_B4B-XH-A_1x04_P2.50mm_Vertical, symbol Connector:Conn_01x04_Pin
- added J6: EXT I/O, Connector_PinHeader_2.54mm:PinHeader_1x04_P2.54mm_Vertical, symbol Connector:Conn_01x04_Pin
- added J7: USB-C 5V IN, Connector_USB:USB_C_Receptacle_GCT_USB4125-xx-x-0190_6P_TopMnt_Horizontal, symbol Connector:USB_C_Receptacle_PowerOnly_6P
- added R13, R14: 2k2, Resistor_SMD:R_0805_2012Metric_Pad1.20x1.40mm_HandSolder, symbol Device:R
- added R15, R16: 1k, Resistor_SMD:R_0805_2012Metric_Pad1.20x1.40mm_HandSolder, symbol Device:R
- added R17: 0R, Resistor_SMD:R_0805_2012Metric_Pad1.20x1.40mm_HandSolder, symbol Device:R
- added R18, R19: 100R, Resistor_SMD:R_0805_2012Metric_Pad1.20x1.40mm_HandSolder, symbol Device:R
- added R20, R21: 4k7, Resistor_SMD:R_0805_2012Metric_Pad1.20x1.40mm_HandSolder, symbol Device:R
- added R22, R23: 5k1, Resistor_SMD:R_0805_2012Metric_Pad1.20x1.40mm_HandSolder, symbol Device:R
- added U3: ISO7721D, Package_SO:SOIC-8_3.9x4.9mm_P1.27mm, symbol Isolator:ISO7721D
- C2: value 100nF -> 10uF 16V X5R; MPN GRM21BR71H104KA01L -> CC0805KRX5R7BB106; Manufacturer Murata -> Yageo
- C3, C5, C6: MPN GRM21BR71H104KA01L -> CL21B104KBCNNNC; Manufacturer Murata -> Samsung Electro-Mechanics
- C4, C7: MPN GRM21BR61C106KE15L -> CC0805KRX5R7BB106; Manufacturer Murata -> Yageo
- C8: MPN GRM21BR71C105KA01L -> GRM219R71E105KA88D
- C9: MPN GRM31CR71E106KA12L -> GRM31CR71E106MA12L
- PS1: value TEM 2-0511 -> TMR 1-0511; footprint sdc_emulator:Traco_TEM2_Single_DIP24 -> Converter_DCDC:Converter_DCDC_TRACO_TMR-1-xxxx_Single_THT; symbol sdc_emulator:TEM2-0511 -> sdc_emulator:TMR1-0511; MPN TEM 2-0511 -> TMR 1-0511
- R10: MPN RN55E2492BB14 -> YR1B24K9CC; Manufacturer Vishay Dale -> TE Connectivity
- R12: MPN RC0805FR-0720KL -> RMCF0805FT20K0; Manufacturer Yageo -> Stackpole Electronics
- R9: MPN RN55E1822BB14 -> YR1B18K2CC; Manufacturer Vishay Dale -> TE Connectivity
Connections:
- net +3V3: now also C10.1, J6.1 (Pin_1), R20.1, R21.1, U3.1 (VCC1)
- net +5V: now also PS1.2 (+Vin), R13.1, R14.1; no longer PS1.1 (+Vin), PS1.24 (+Vin)
- net +5V_IN: now also J7.A9 (VBUS), J7.B9 (VBUS)
- net COIL_N: now also D4.1 (K)
- net GND: now also PS1.1 (-Vin), C10.2, D3.1 (K), J6.4 (Pin_4), J7.A12 (GND), J7.B12 (GND), J7.S1 (SHIELD), R22.2, R23.2, U3.4 (GND1); no longer PS1.12 (-Vin), PS1.13 (-Vin)
- net GND_ISO: now also PS1.6 (-Vout), C11.2, J5.1 (Pin_1), U3.5 (GND2); no longer PS1.10 (-Vout), PS1.15 (-Vout)
- net VDD_ISO: now also PS1.4 (+Vout), C11.1, R17.2, U3.8 (VCC2); no longer PS1.11 (+Vout), PS1.14 (+Vout)
- net SVC_RX: now reaches J1.6 (Pin_6)
- net SVC_RX: now also U3.2 (OUTA)
- net SVC_TX: now reaches J1.7 (Pin_7)
- net SVC_TX: now also U3.3 (INB)
- net EXT_IO1: now reaches J2.4 (Pin_4)
- net EXT_IO1: now also R19.2, R21.2
- net EXT_IO2: now reaches J2.5 (Pin_5)
- net EXT_IO2: now also R18.2, R20.2
- new net EXT_IO1_H: J6.3 (Pin_3), R19.1
- new net EXT_IO2_H: J6.2 (Pin_2), R18.1
- new net LED_PWR: D3.2 (A), R13.2
- new net LED_REL: D4.2 (A), R14.2
- new net SVC_5V: J5.4 (Pin_4), R17.1
- new net SVC_RX_EXT: J5.2 (Pin_2), R15.1
- new net SVC_RX_ISO: R15.2, U3.7 (INA)
- new net SVC_TX_EXT: J5.3 (Pin_3), R16.1
- new net SVC_TX_ISO: R16.2, U3.6 (OUTB)
- new net USB_CC1: J7.A5 (CC1), R22.1
- new net USB_CC2: J7.B5 (CC2), R23.1
- no-connect marks 34 -> 30
Other:
- note added: "DevKit: ESP32-S3-DevKitC-1 (N16R8 clone), header rows 25.1 mm apart (measured). GPIO4 = RELAY_EN (ESPHome restore_mode ALWAYS_OFF), GPIO5 = RELAY_SENSE (LOW = coil on), GPIO8 = SDA, GPIO9 = SCL, GPIO6 = service RX, GPIO7 = service TX (UART), GPIO1/GPIO2 = expansion header J6."
- note added: "PS1 TMR 1-0511: regulated, no minimum load. Pin 3/5 absent: 5.08 mm between +Vin (2) and +Vout (4)."
- note added: "SDC service port (J5): UART at 5 V logic, isolated by U3. Pinout of the SDC socket is not yet known: J5-2 RX must go to the SDC's TX, J5-3 TX to the SDC's RX. J5-1 is GND_ISO (= SDC X5 ground): only connect if the port GND is the same potential. R17 (0R): remove if the SDC port has its own 5 V supply pin."
- note removed: "DevKit: ESP32-S3-DevKitC-1 (N16R8 clone), header rows 25.1 mm apart (measured). GPIO4 = RELAY_EN (ESPHome restore_mode ALWAYS_OFF), GPIO5 = RELAY_SENSE (LOW = coil on), GPIO8 = SDA, GPIO9 = SCL."
- note removed: "R8 is DNP: fit only if TEM no-load output > 5.4 V."
